File: BQ24257/BQ24257.kicad_pcb (KiCad board)
At the start: 4 copper layers, 57.4 x 51.4 mm, 68 parts, among them IC1 LTC1982ES6#TRMPBF, IC2 LTC3113EDHD#TRPBF, J3 UPDI, J4 NTC, Q2 SQS201CENW-T1_GE3, Q3 IRLML6401, Q4 SUD09P10-195, U1 BQ24257RGET, U2 AD5280, U3 AMS1117-3.3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

Commit message: passed DRC
Parts:
- moved Cpmid1 1.18 mm to (55.2, 114.8)
- moved Cboot1 1.03 mm to (55.8, 115.9)
- moved Lo1 0.28 mm to (51.8, 112.4)
Routing:
- net VIN: track 27.3 -> 36.0 mm, vias 4 -> 5
- net GND: track 78.6 -> 83.1 mm, vias 79 -> 75
- net VBAT: track 77.5 -> 79.6 mm
- net U/D: track 51.8 -> 53.5 mm
- net Net-(U1-BOOT): track 1.39 -> 2.49 mm
- net Net-(Cboot1-Pad2): track 7.91 -> 8.84 mm
- net VSYS: track 165.4 -> 166.3 mm
Other:
- board text added: "BQ24257 MPPT TEST KIT"
- board text added: "lucy moglia, 11/8/24"
